File: hardware/servo.kicad_pcb (KiCad board)
At the start: 2 copper layers, 40 x 40 mm, 9 parts, among them P1 CON-SENSOR2, P2 CONN_01X02, U1 pin_array_6x3, U2 pin_array_6x3, U3 DRILL, U4 DRILL, U5 DRILL, U6 DRILL, U7 XMC1XXX48

Commit message: pcb design
Parts:
- added C1: 10uF, kicad-libraries:C0805, F.Cu at (151.9, 89.0)
- added C10: 100nF, kicad-libraries:C0603, F.Cu at (140.5, 102.8)
- added C11: 100nF, kicad-libraries:C0603, F.Cu at (167.1, 102.3)
- added C12: 10uF, kicad-libraries:C0805, F.Cu at (154.5, 90.0)
- added C2: 1uF, kicad-libraries:C0603F, F.Cu at (151.9, 90.5)
- added C3: 100nF, kicad-libraries:C0603F, F.Cu at (175.8, 107.3)
- added C4: 100nF, kicad-libraries:C0603F, F.Cu at (143.1, 96.4)
- added C5: 100nF, kicad-libraries:C0603F, F.Cu at (144.2, 99.1)
- added C6: 220nF, kicad-libraries:C0603F, F.Cu at (144.4, 96.4)
- added C7: 220pF, kicad-libraries:C0402F, F.Cu at (146.3, 89.7)
- added C8: 10pF, kicad-libraries:C0603F, F.Cu at (157.5, 100.7)
- added C9: 10pF, kicad-libraries:C0603F, F.Cu at (157.5, 95.3)
- added D1: Z12V, kicad-libraries:SOD-123, F.Cu at (148.2, 109.3)
- added D3: blue, kicad-libraries:D0603E, F.Cu at (160.4, 84.4)
- added P3: DEBUG, kicad-libraries:DEBUG_PAD, F.Cu at (176.1, 97.5)
- added P4: black, kicad-libraries:OQ_2P, F.Cu at (150.0, 114.3)
- added Q1: FDS8449, kicad-libraries:SOIC-8-MOSFET, F.Cu at (151.7, 108.5)
- added R1: 1k, kicad-libraries:R0603F, F.Cu at (160.4, 85.8)
- added R10: 0R1, kicad-libraries:R0805E, F.Cu at (165.8, 115.0)
- added R11: 0R1, kicad-libraries:R0805E, F.Cu at (163.3, 115.0)
- added R12: 0R1, kicad-libraries:R0805E, F.Cu at (160.8, 115.0)
- added R13: 0R1, kicad-libraries:R0805E, F.Cu at (158.2, 115.0)
- added R16: 100k, kicad-libraries:R0603F, F.Cu at (147.4, 105.7)
- added R2: 10k, kicad-libraries:R0603F, F.Cu at (146.4, 110.8)
- added R3: 1k, kicad-libraries:R0603F, F.Cu at (146.4, 107.9)
- added R4: 0R1, kicad-libraries:R0805E, F.Cu at (141.8, 115.0)
- added R5: 0R1, kicad-libraries:R0805E, F.Cu at (139.2, 115.0)
- added R6: 0R1, kicad-libraries:R0805E, F.Cu at (158.3, 115.0)
- added R6: 0R1, kicad-libraries:R0805E, F.Cu at (136.7, 115.0)
- added R7: 0R1, kicad-libraries:R0805E, F.Cu at (134.2, 115.0)
- added R8: 0R1, kicad-libraries:R0805E, F.Cu at (131.7, 115.0)
- added R9: 0R1, kicad-libraries:R0805E, F.Cu at (168.3, 115.0)
- added RP1: 82, kicad-libraries:4X0402, F.Cu at (148.1, 89.7)
- added U8: Con_Servo_5x, kicad-libraries:pin_array_5x3, F.Cu at (136.7, 109.0)
- added U9: Con_Servo_5x, kicad-libraries:pin_array_5x3, F.Cu at (163.3, 109.0)
- added X1: 16MHz, kicad-libraries:CRYSTAL_3225, F.Cu at (157.5, 98.0)
- P2: value CONN_01X02 -> BOOT; footprint kicad-libraries:OQ_2P -> kicad-libraries:SolderJumper
- U1: value pin_array_6x3 -> XMC1404; footprint kicad-libraries:pin_array_6x3 -> kicad-libraries:QFN48-EP2
- U2: value pin_array_6x3 -> DRILL; footprint kicad-libraries:pin_array_6x3 -> kicad-libraries:DRILL_NP
- U6: value DRILL -> 74HC245; footprint kicad-libraries:DRILL_NP -> kicad-libraries:TSSOP20
- U7: value XMC1XXX48 -> 74HC245; footprint kicad-libraries:QFN48-EP2 -> kicad-libraries:TSSOP20
- moved U4 49.5 mm to (132.5, 120.0)
- moved P2 36.7 mm to (175.9, 99.8)
- moved U3 35.0 mm to (167.5, 120.0)
- moved U5 35.0 mm to (167.5, 85.0)
- moved U2 34.5 mm to (132.5, 85.0)
- moved U7 26.6 mm to (163.0, 100.3), turned to 180 degrees
- moved U6 15.8 mm to (136.4, 100.3), turned to 180 degrees
- moved U1 6.23 mm to (150.0, 97.5), turned to 180 degrees
- moved P1 0.10 mm to (150.0, 82.6)
Connections:
- P1 pad 1: Net-(P1-Pad1) -> +5V
- P1 pad 2: Net-(P1-Pad2) -> GND
- P1 pad 3: Net-(P1-Pad3) -> VCC
- P1 pad EP: Net-(P1-PadEP) -> GND
- P2 pad 1: Net-(P2-Pad1) -> GND
- U1 pad 10: Net-(U1-Pad10) -> CUR-SERVO-7
- U1 pad 11: Net-(U1-Pad11) -> CUR-SERVO-8
- U1 pad 12: Net-(U1-Pad12) -> CUR-SERVO-9
- U1 pad 13: Net-(U1-Pad13) -> V-EXT
- U1 pad 17: Net-(U1-Pad17) -> GND
- U1 pad 18: Net-(U1-Pad18) -> VCC
- U1 pad 2: Net-(U1-Pad2) -> Net-(P2-Pad2)
- U1 pad 3: Net-(U1-Pad3) -> CUR-SERVO-0
- U1 pad 4: Net-(U1-Pad4) -> CUR-SERVO-1
- U1 pad 5: Net-(U1-Pad5) -> CUR-SERVO-2
- U1 pad 6: Net-(U1-Pad6) -> CUR-SERVO-3
- U1 pad 7: Net-(U1-Pad7) -> CUR-SERVO-4
- U1 pad 8: Net-(U1-Pad8) -> CUR-SERVO-5
- U1 pad 9: Net-(U1-Pad9) -> CUR-SERVO-6
- U7 pad 1: (no net) -> +5V
- U7 pad 10: (no net) -> GND
- U7 pad 11: (no net) -> Net-(U7-Pad11)
- U7 pad 12: (no net) -> Net-(U7-Pad12)
- U7 pad 13: (no net) -> Net-(U7-Pad13)
- U7 pad 14: (no net) -> Net-(U7-Pad14)
- U7 pad 15: (no net) -> Net-(U7-Pad15)
- U7 pad 16: (no net) -> Net-(U7-Pad16)
- U7 pad 19: Net-(U7-Pad19) -> GND
- U7 pad 2: (no net) -> PWM-SERVO-5
- U7 pad 20: (no net) -> +5V
- U7 pad 3: (no net) -> PWM-SERVO-6
- U7 pad 4: (no net) -> PWM-SERVO-7
- U7 pad 5: (no net) -> PWM-SERVO-8
- U7 pad 6: (no net) -> PWM-SERVO-9
- U7 pad 7: (no net) -> GND
- U7 pad 8: (no net) -> GND
- U7 pad 9: (no net) -> GND
Routing:
- net Net-(P4-Pad1): track 0.00 -> 62.9 mm
- net GND: track 0.00 -> 26.0 mm, vias 0 -> 44
- net PWM-SERVO-4: track 0.00 -> 21.7 mm
- net PWM-SERVO-3: track 0.00 -> 19.7 mm
- net PWM-SERVO-2: track 0.00 -> 18.2 mm
- net PWM-SERVO-1: track 0.00 -> 17.7 mm
- net PWM-SERVO-5: track 0.00 -> 16.2 mm
- net PWM-SERVO-6: track 0.00 -> 15.5 mm
- net PWM-SERVO-0: track 0.00 -> 15.2 mm
- net PWM-SERVO-7: track 0.00 -> 14.9 mm
- net PWM-SERVO-9: track 0.00 -> 12.8 mm
- net PWM-SERVO-8: track 0.00 -> 12.8 mm
- net Net-(C8-Pad1): track 0.00 -> 6.97 mm
- net VCC: track 0.00 -> 6.04 mm
- net Net-(U6-Pad14): track 0.00 -> 5.84 mm
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- added copper zone on F.Cu, net GND
- added copper zone on GND, net GND
- added copper zone on VCC, net Net-(P4-Pad1)
- added copper zone on F.Cu, net Net-(P4-Pad2)
Other:
- copper layers 2 -> 4
- rule trace_min: 0.2 -> 0.1
- rule via_min_drill: 0.3 -> 0.2

Commit message: pcb design
Parts:
- moved C3 21.6 mm to (155.4, 100.2), turned to 270 degrees
- moved P2 20.7 mm to (156.3, 93.4), turned to 270 degrees
- moved P3 18.5 mm to (158.0, 93.7)
- moved C5 4.96 mm to (146.9, 103.2)
- moved C12 2.49 mm to (156.3, 88.3), turned to 0 degrees
- moved C8 0.50 mm to (158.0, 100.7)
- moved C9 0.50 mm to (158.0, 95.3)
- moved X1 0.50 mm to (158.0, 98.0)
- moved D1 0.40 mm to (148.2, 109.7)
- moved R2 0.40 mm to (146.4, 111.2)
- moved R16 0.40 mm to (147.4, 106.1)
- moved R3 0.40 mm to (146.4, 108.3)
- moved C10 0.39 mm to (140.6, 102.4)
- moved C1 0.20 mm to (151.9, 89.2)
- moved C2 0.20 mm to (151.9, 90.7)
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Connections:
- U1 pad 1: Net-(U1-Pad1) -> Net-(R1-Pad1)
- U1 pad 10: CUR-SERVO-7 -> CUR-SERVO-2
- U1 pad 11: CUR-SERVO-8 -> CUR-SERVO-3
- U1 pad 12: CUR-SERVO-9 -> CUR-SERVO-4
- U1 pad 2: Net-(P2-Pad2) -> Net-(U1-Pad2)
- U1 pad 29: PWM-SERVO-0 -> PWM-SERVO-1
- U1 pad 3: CUR-SERVO-0 -> CUR-SERVO-5
- U1 pad 30: PWM-SERVO-1 -> PWM-SERVO-4
- U1 pad 35: PWM-SERVO-4 -> PWM-SERVO-0
- U1 pad 4: CUR-SERVO-1 -> CUR-SERVO-6
- U1 pad 48: Net-(R1-Pad1) -> Net-(P2-Pad2)
- U1 pad 5: CUR-SERVO-2 -> CUR-SERVO-7
- U1 pad 6: CUR-SERVO-3 -> CUR-SERVO-8
- U1 pad 7: CUR-SERVO-4 -> CUR-SERVO-9
- U1 pad 8: CUR-SERVO-5 -> CUR-SERVO-0
- U1 pad 9: CUR-SERVO-6 -> CUR-SERVO-1
Routing:
- net +5V: track 0.00 -> 70.1 mm
- net GND: track 26.0 -> 64.9 mm, vias 44 -> 72
- net S-MOSI: track 0.00 -> 17.6 mm
- net S-CLK: track 0.00 -> 16.9 mm
- net VCC: track 6.04 -> 21.1 mm, vias 0 -> 7
- net S-CS: track 0.00 -> 14.1 mm, vias 0 -> 2
- net Net-(R1-Pad1): track 0.00 -> 13.2 mm, vias 0 -> 2
- net S-MISO: track 0.00 -> 10.5 mm, vias 0 -> 2
- net Net-(P3-Pad1): track 0.00 -> 5.05 mm
- net Net-(P4-Pad1): track 62.9 -> 67.7 mm
- net Net-(P2-Pad2): track 0.00 -> 3.38 mm
- net PWM-SERVO-4: track 21.7 -> 18.4 mm, vias 0 -> 2
- net PWM-SERVO-1: track 17.7 -> 15.1 mm, vias 0 -> 2
- net PWM-SERVO-9: track 12.8 -> 11.2 mm, vias 0 -> 2
- net Net-(D3-Pad2): track 0.00 -> 1.44 mm
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- added copper zone on VCC, net VCC
- removed copper zone on VCC, net Net-(P4-Pad1)

Commit message: pcb design
Parts:
- removed the R6 at (158.3, 115.0)
- moved RP1 4.80 mm to (143.8, 91.7)
- moved C7 4.75 mm to (142.0, 91.7)
Connections:
- U1 pad 11: CUR-SERVO-3 -> CUR-SERVO-1
- U1 pad 12: CUR-SERVO-4 -> CUR-SERVO-0
- U1 pad 3: CUR-SERVO-5 -> CUR-SERVO-9
- U1 pad 4: CUR-SERVO-6 -> CUR-SERVO-8
- U1 pad 6: CUR-SERVO-8 -> CUR-SERVO-6
- U1 pad 7: CUR-SERVO-9 -> CUR-SERVO-5
- U1 pad 8: CUR-SERVO-0 -> CUR-SERVO-4
- U1 pad 9: CUR-SERVO-1 -> CUR-SERVO-3
Routing:
- net CUR-SERVO-5: track 2.47 -> 43.1 mm, vias 0 -> 1
- net CUR-SERVO-4: track 2.47 -> 42.3 mm, vias 0 -> 1
- net CUR-SERVO-6: track 2.46 -> 39.7 mm, vias 0 -> 1
- net CUR-SERVO-3: track 2.46 -> 38.9 mm, vias 0 -> 1
- net CUR-SERVO-7: track 2.46 -> 36.4 mm, vias 0 -> 1
- net CUR-SERVO-2: track 2.46 -> 35.6 mm, vias 0 -> 1
- net CUR-SERVO-8: track 2.46 -> 33.0 mm, vias 0 -> 1
- net CUR-SERVO-1: track 2.46 -> 32.6 mm, vias 0 -> 1
- net V-EXT: track 1.40 -> 25.6 mm, vias 0 -> 3
- net CUR-SERVO-9: track 2.47 -> 26.3 mm, vias 0 -> 1
- net CUR-SERVO-0: track 2.47 -> 25.8 mm, vias 0 -> 1
- net Net-(P1-Pad4): track 2.61 -> 8.09 mm
- net Net-(P1-Pad5): track 2.09 -> 7.48 mm
- net Net-(C7-Pad1): track 3.10 -> 7.96 mm
- net Net-(P1-Pad6): track 2.07 -> 6.69 mm
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- added copper zone on F.Cu, net VCC

Commit message: final prototype design, drc check, silkscreen added
Parts:
- added G***: LOGO, kicad-libraries:Logo_CoMCU, B.Cu at (157.5, 101.5)
- added G***: LOGO, kicad-libraries:Logo_31x31, F.Cu at (136.4, 91.6)
- added VAL: WEEE_7mm, kicad-libraries:WEEE_7mm, B.Cu at (150.0, 102.0)
- added VAL: CE_5mm, kicad-libraries:CE_5mm, B.Cu at (143.0, 101.5)
- moved R1 0.88 mm to (160.7, 86.6)
- moved D3 0.88 mm to (160.7, 85.2)
Routing:
- net CUR-SERVO-9: track 26.3 -> 27.5 mm
- net CUR-SERVO-4: track 42.3 -> 43.2 mm
- net CUR-SERVO-8: track 33.0 -> 33.7 mm
Other:
- net class Default: clearance 0.2 -> 0.15; trace_width 0.25 -> 0.2; via_dia 0.8 -> 0.55; via_drill 0.4 -> 0.25
- rule trace_clearance: 0.2 -> 0.15
- board text added: "+"
- board text added: "-"
- board text added: "0"
- board text added: "1"
- board text added: "2"
- board text added: "3"
- board text added: "4"
- board text added: "5"
- board text added: "6"
- board text added: "7"
- board text added: "8"
- board text added: "9"
- board text added: "Input max 27V"
- board text added: "Servo 1.0"
- board text added: "Status"
- board text added: "tinkerforge.com"

Commit message: ready for prototype
Connections:
- R10 pad 1: CUR-SERVO-6 -> CUR-SERVO-8
- R12 pad 1: CUR-SERVO-8 -> CUR-SERVO-6
- R13 pad 1: CUR-SERVO-9 -> CUR-SERVO-5
- R4 pad 1: CUR-SERVO-0 -> CUR-SERVO-4
- R5 pad 1: CUR-SERVO-1 -> CUR-SERVO-3
- R7 pad 1: CUR-SERVO-3 -> CUR-SERVO-1
- R8 pad 1: CUR-SERVO-4 -> CUR-SERVO-0
- R9 pad 1: CUR-SERVO-5 -> CUR-SERVO-9
- U1 pad 11: CUR-SERVO-1 -> CUR-SERVO-3
- U1 pad 12: CUR-SERVO-0 -> CUR-SERVO-4
- U1 pad 29: PWM-SERVO-1 -> PWM-SERVO-3
- U1 pad 3: CUR-SERVO-9 -> CUR-SERVO-5
- U1 pad 30: PWM-SERVO-4 -> PWM-SERVO-0
- U1 pad 32: PWM-SERVO-3 -> PWM-SERVO-1
- U1 pad 35: PWM-SERVO-0 -> PWM-SERVO-4
- U1 pad 36: PWM-SERVO-5 -> PWM-SERVO-9
- U1 pad 39: PWM-SERVO-6 -> PWM-SERVO-8
- U1 pad 4: CUR-SERVO-8 -> CUR-SERVO-6
- U1 pad 43: PWM-SERVO-9 -> PWM-SERVO-5
- U1 pad 46: PWM-SERVO-8 -> PWM-SERVO-6
- U1 pad 6: CUR-SERVO-6 -> CUR-SERVO-8
- U1 pad 7: CUR-SERVO-5 -> CUR-SERVO-9
- U1 pad 8: CUR-SERVO-4 -> CUR-SERVO-0
- U1 pad 9: CUR-SERVO-3 -> CUR-SERVO-1
- U6 pad 2: PWM-SERVO-0 -> PWM-SERVO-4
- U6 pad 3: PWM-SERVO-1 -> PWM-SERVO-3
- U6 pad 5: PWM-SERVO-3 -> PWM-SERVO-1
- U6 pad 6: PWM-SERVO-4 -> PWM-SERVO-0
- U7 pad 2: PWM-SERVO-5 -> PWM-SERVO-9
- U7 pad 3: PWM-SERVO-6 -> PWM-SERVO-8
- U7 pad 5: PWM-SERVO-8 -> PWM-SERVO-6
- U7 pad 6: PWM-SERVO-9 -> PWM-SERVO-5
- U8 pad A1: CUR-SERVO-4 -> CUR-SERVO-0
- U8 pad B1: CUR-SERVO-3 -> CUR-SERVO-1
- U8 pad D1: CUR-SERVO-1 -> CUR-SERVO-3
- U8 pad E1: CUR-SERVO-0 -> CUR-SERVO-4
- U9 pad A1: CUR-SERVO-9 -> CUR-SERVO-5
- U9 pad B1: CUR-SERVO-8 -> CUR-SERVO-6
- U9 pad D1: CUR-SERVO-6 -> CUR-SERVO-8
- U9 pad E1: CUR-SERVO-5 -> CUR-SERVO-9
Routing:
- net CUR-SERVO-4: track 43.2 -> 26.2 mm
- net CUR-SERVO-0: track 26.2 -> 43.2 mm
- net CUR-SERVO-9: track 27.5 -> 43.3 mm
- net CUR-SERVO-5: track 43.3 -> 27.5 mm
- net CUR-SERVO-3: track 39.2 -> 32.7 mm
- net CUR-SERVO-1: track 32.7 -> 39.2 mm
- net CUR-SERVO-8: track 33.7 -> 40.0 mm
- net CUR-SERVO-6: track 40.0 -> 33.7 mm
- net PWM-SERVO-9: track 11.2 -> 17.3 mm
- net PWM-SERVO-5: track 17.3 -> 11.2 mm
- net PWM-SERVO-3: track 18.5 -> 14.3 mm
- net PWM-SERVO-1: track 14.3 -> 18.5 mm
- net PWM-SERVO-8: track 11.7 -> 15.6 mm
- net PWM-SERVO-6: track 15.6 -> 11.7 mm
- net PWM-SERVO-4: track 18.4 -> 16.4 mm
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Other:
- board text added: "Servo 2.0"
- board text added: "Servo Voltage"
- board text added: "Voltage is directly applied to servo!"
- board text removed: "Input max 27V"
- board text removed: "Servo 1.0"

Commit message: ordered version
Other:
- rule pad_to_mask_clearance: 0.051 -> 0
Changed lines of the file:
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@@
-(kicad_pcb (version 20171130) (host pcbnew 5.1.4-e60b266~84~ubuntu19.04.1)
+(kicad_pcb (version 20171130) (host pcbnew 5.1.4-e60b266~84~ubuntu18.04.1)
   (general
     (thickness 1.6)
@@
     (pad_size 1.524 1.524)
     (pad_drill 0.762)
-    (pad_to_mask_clearance 0.051)
-    (solder_mask_min_width 0.25)
+    (pad_to_mask_clearance 0)
     (aux_axis_origin 130 82.5)
     (grid_origin 130 82.5)
@@
     (pcbplotparams
       (layerselection 0x010fc_ffffffff)
-      (usegerberextensions false)
+      (usegerberextensions true)
       (usegerberattributes false)
       (usegerberadvancedattributes false)
@@
       (psnegative false)
       (psa4output false)
-      (plotreference true)
-      (plotvalue true)
+      (plotreference false)
+      (plotvalue false)
       (plotinvisibletext false)
       (padsonsilk false)
-      (subtractmaskfromsilk false)
+      (subtractmaskfromsilk true)
       (outputformat 1)
       (mirror false)
-      (drillshape 1)
+      (drillshape 0)
       (scaleselection 1)
-      (outputdirectory ""))
+      (outputdirectory "pcb/"))
   )
   (net 0 "")
